File: Tri 2/ECEN405/Lab 5/schematic/Lab 5.sch (KiCad schematic (older format))
At the start: 11 parts

Commit message: updated 405
Connections:
- net +15V: now also U?.1 (VCC)
- net GND: no longer U?.1 (VCC)
Other:
- note added: "+"
- note added: "-"
- moved on the sheet: C?
Changed lines of the file:
@@
 L Device:C_Small C?
 U 1 1 610FA5FA
-P 1400 1625
-F 0 "C?" H 1492 1671 50  0000 L CNN
-F 1 "10u 50V" H 1492 1580 50  0000 L CNN
-F 2 "" H 1400 1625 50  0001 C CNN
-F 3 "~" H 1400 1625 50  0001 C CNN
-	1    1400 1625
-	1    0    0    -1
-$EndComp
-Wire Wire Line
-	1400 1725 1400 1875
-Connection ~ 1400 2075
+P 1400 1975
+F 0 "C?" H 1200 1900 50  0000 L CNN
+F 1 "10u 50V" H 1025 1825 50  0000 L CNN
+F 2 "" H 1400 1975 50  0001 C CNN
+F 3 "~" H 1400 1975 50  0001 C CNN
+	1    1400 1975
+	1    0    0    -1
+$EndComp
 Wire Wire Line
 	1600 1875 1400 1875
-Connection ~ 1400 1875
-Wire Wire Line
-	1400 1875 1400 2075
 Wire Wire Line
 	1600 1975 1050 1975
@@
 $EndComp
 Wire Wire Line
-	1400 1525 1400 1300
-Wire Wire Line
 	2075 1300 1400 1300
 Connection ~ 1400 1300
@@
 	5550 2850 4975 2850
 Connection ~ 4975 2850
+Wire Wire Line
+	1400 1300 1400 1875
+Connection ~ 1400 1875
+Connection ~ 1400 2075
+Text Notes 5625 2425 0    50   ~ 0
+-
+Text Notes 5625 2850 0    50   ~ 0
++
 $EndSCHEMATC

Commit message: ECEN 405 lab 5
Parts:
- gave numbers to parts that had none: 11
Other:
- note added: "V_out"
Changed lines of the file:
@@
 $EndDescr
 $Comp
-L IR2117SPBF:IR2117SPBF U?
+L IR2117SPBF:IR2117SPBF U1
 U 1 1 610F7041
 P 2250 2025
-F 0 "U?" H 2250 2575 60  0000 C CNN
+F 0 "U1" H 2250 2575 60  0000 C CNN
 F 1 "IR2117SPBF" H 2250 2475 60  0000 C CNN
 F 2 "SOIC8_INF" H 3050 2265 60  0001 C CNN
@@
 $EndComp
 $Comp
-L power:+15V #PWR?
+L power:+15V #PWR01
 U 1 1 610F8D3B
 P 1400 1225
-F 0 "#PWR?" H 1400 1075 50  0001 C CNN
+F 0 "#PWR01" H 1400 1075 50  0001 C CNN
 F 1 "+15V" H 1415 1398 50  0000 C CNN
 F 2 "" H 1400 1225 50  0001 C CNN
@@
 $EndComp
 $Comp
-L power:GND #PWR?
+L power:GND #PWR02
 U 1 1 610F97B6
 P 1400 2375
-F 0 "#PWR?" H 1400 2125 50  0001 C CNN
+F 0 "#PWR02" H 1400 2125 50  0001 C CNN
 F 1 "GND" H 1405 2202 50  0000 C CNN
 F 2 "" H 1400 2375 50  0001 C CNN
@@
 	1400 2075 1600 2075
 $Comp
-L Device:C_Small C?
+L Device:C_Small C1
 U 1 1 610FA5FA
 P 1400 1975
-F 0 "C?" H 1200 1900 50  0000 L CNN
+F 0 "C1" H 1200 1900 50  0000 L CNN
 F 1 "10u 50V" H 1025 1825 50  0000 L CNN
 F 2 "" H 1400 1975 50  0001 C CNN
@@
 control
 $Comp
-L Device:D D?
+L Device:D D1
 U 1 1 610FED8B
 P 2225 1300
-F 0 "D?" H 2225 1083 50  0000 C CNN
+F 0 "D1" H 2225 1083 50  0000 C CNN
 F 1 "D" H 2225 1174 50  0000 C CNN
 F 2 "" H 2225 1300 50  0001 C CNN
@@
 	2975 1875 2850 1875
 $Comp
-L Device:C_Small C?
+L Device:C_Small C2
 U 1 1 611008BD
 P 2975 1975
-F 0 "C?" H 3067 2021 50  0000 L CNN
+F 0 "C2" H 3067 2021 50  0000 L CNN
 F 1 "10u 50V" H 3067 1930 50  0000 L CNN
 F 2 "" H 2975 1975 50  0001 C CNN
@@
 	2975 2075 2850 2075
 $Comp
-L Device:R_Small R?
+L Device:R_Small R1
 U 1 1 61102557
 P 3650 1975
-F 0 "R?" V 3454 1975 50  0000 C CNN
+F 0 "R1" V 3454 1975 50  0000 C CNN
 F 1 "10" V 3545 1975 50  0000 C CNN
 F 2 "" H 3650 1975 50  0001 C CNN
@@
 	3550 1975 2850 1975
 $Comp
-L Device:Q_NMOS_GDS Q?
+L Device:Q_NMOS_GDS Q1
 U 1 1 6110323C
 P 4050 1975
-F 0 "Q?" H 4254 2021 50  0000 L CNN
+F 0 "Q1" H 4254 2021 50  0000 L CNN
 F 1 "Q_NMOS_GDS" H 4254 1930 50  0000 L CNN
 F 2 "" H 4250 2075 50  0001 C CNN
@@
 Connection ~ 2975 2075
 $Comp
-L power:VCC #PWR?
+L power:VCC #PWR03
 U 1 1 61104A91
-P 4150 1200
-F 0 "#PWR?" H 4150 1050 50  0001 C CNN
-F 1 "VCC" H 4165 1373 50  0000 C CNN
-F 2 "" H 4150 1200 50  0001 C CNN
-F 3 "" H 4150 1200 50  0001 C CNN
-	1    4150 1200
-	1    0    0    -1
-$EndComp
-Wire Wire Line
-	4150 1200 4150 1275
-$Comp
-L Device:C_Small C?
+P 4150 1225
+F 0 "#PWR03" H 4150 1075 50  0001 C CNN
+F 1 "VCC" H 4165 1398 50  0000 C CNN
+F 2 "" H 4150 1225 50  0001 C CNN
+F 3 "" H 4150 1225 50  0001 C CNN
+	1    4150 1225
+	1    0    0    -1
+$EndComp
+Wire Wire Line
+	4150 1225 4150 1275
+$Comp
+L Device:C_Small C3
 U 1 1 611054E7
 P 4325 1375
-F 0 "C?" H 4417 1421 50  0000 L CNN
+F 0 "C3" H 4417 1421 50  0000 L CNN
 F 1 "10u 50V" H 4417 1330 50  0000 L CNN
 F 2 "" H 4325 1375 50  0001 C CNN
@@
 	4150 1275 4150 1775
 $Comp
-L power:GND #PWR?
+L power:GND #PWR05
 U 1 1 61105FCF
 P 4325 1550
-F 0 "#PWR?" H 4325 1300 50  0001 C CNN
+F 0 "#PWR05" H 4325 1300 50  0001 C CNN
 F 1 "GND" H 4330 1377 50  0000 C CNN
 F 2 "" H 4325 1550 50  0001 C CNN
@@
 	4325 1475 4325 1550
 $Comp
-L Device:L L?
+L Device:L L1
 U 1 1 61107B8B
 P 4150 2625
-F 0 "L?" H 4202 2671 50  0000 L CNN
+F 0 "L1" H 4202 2671 50  0000 L CNN
 F 1 "4m" H 4202 2580 50  0000 L CNN
 F 2 "" H 4150 2625 50  0001 C CNN
@@
 Connection ~ 4150 2375
 $Comp
-L power:GND #PWR?
+L power:GND #PWR04
 U 1 1 61108ABD
 P 4150 2900
-F 0 "#PWR?" H 4150 2650 50  0001 C CNN
+F 0 "#PWR04" H 4150 2650 50  0001 C CNN
 F 1 "GND" H 4155 2727 50  0000 C CNN
 F 2 "" H 4150 2900 50  0001 C CNN
@@
 	4150 2775 4150 2850
 $Comp
-L Device:D D?
+L Device:D D2
 U 1 1 611097C5
 P 4575 2375
-F 0 "D?" H 4575 2592 50  0000 C CNN
+F 0 "D2" H 4575 2592 50  0000 C CNN
 F 1 "D" H 4575 2501 50  0000 C CNN
 F 2 "" H 4575 2375 50  0001 C CNN
@@
 	4975 2375 4975 2525
 $Comp
-L Device:CP_Small C?
+L Device:CP_Small C4
 U 1 1 6110C7BD
 P 4975 2625
-F 0 "C?" H 4887 2579 50  0000 R CNN
+F 0 "C4" H 4887 2579 50  0000 R CNN
 F 1 "100u 50V" H 4887 2670 50  0000 R CNN
 F 2 "" H 4975 2625 50  0001 C CNN
@@
 	4150 2850 4150 2900
 $Comp
-L Device:R_Small R?
+L Device:R_Small R2
 U 1 1 611126B7
 P 5550 2625
-F 0 "R?" H 5609 2671 50  0000 L CNN
+F 0 "R2" H 5609 2671 50  0000 L CNN
 F 1 "500" H 5609 2580 50  0000 L CNN
 F 2 "" H 5550 2625 50  0001 C CNN
@@
 Connection ~ 1400 1875
 Connection ~ 1400 2075
-Text Notes 5625 2425 0    50   ~ 0
+Text Notes 5625 2425 0    50   ~ 10
 -
-Text Notes 5625 2850 0    50   ~ 0
+Text Notes 5625 2850 0    50   ~ 10
 +
+Text Notes 5800 2650 0    50   ~ 10
+V_out
 $EndSCHEMATC
